Commit message: metal hip link addition

File: bogobot_rviz/urdf/humanoid_links.xacro (robot description, xacro)
@@ -84,3 +84,19 @@
 		</link>
 	</xacro:macro>
+	<xacro:macro name="hip_metal_link" params="name x y z row pitch yaw">
+		<link name="${name}">
+			<collision>
+                		<origin xyz="${x} ${y} ${z}" rpy="${row} ${pitch} ${yaw}"  />
+                		<geometry>
+                    			<mesh filename="package://bogobot_rviz/meshes/metal_cadera_b4.STL" scale="0.001 0.001 0.001"/>
+                		</geometry>
+            		</collision>
+			<visual>
+                		<origin xyz="${x} ${y} ${z}" rpy="${row} ${pitch} ${yaw}" />
+                		<geometry>
+                    			<mesh filename="package://bogobot_rviz/meshes/metal_cadera_b4.STL" scale="0.001 0.001 0.001"/>
+                		</geometry>
+            		</visual>
+		</link>
+	</xacro:macro>
 </robot>

File: bogobot_rviz/urdf/humanoid_main.urdf (robot description, URDF)
Before this commit: robot Bogobot_V1, 7 links, 6 joints
Links:
- added link link_left_hip_metal; collision mesh filename=package://bogobot_rviz/meshes/metal_cadera_b4.STL scale=0.001 0.001 0.001; visual mesh filename=package://bogobot_rviz/meshes/metal_cadera_b4.STL scale=0.001 0.001 0.001
- added link link_right_hip_metal; collision mesh filename=package://bogobot_rviz/meshes/metal_cadera_b4.STL scale=0.001 0.001 0.001; visual mesh filename=package://bogobot_rviz/meshes/metal_cadera_b4.STL scale=0.001 0.001 0.001
Joints:
- added joint q7: type revolute, parent chest, child link_right_hip_metal, origin xyz=0 0.055 0.3825 rpy=0 0 0, axis 1 0 0, limit lower=-6.283185307179586 upper=6.283185307179586 effort=2.5 velocity=5.76
- added joint q8: type revolute, parent chest, child link_left_hip_metal, origin xyz=0 -0.055 0.3825 rpy=0 0 0, axis 1 0 0, limit lower=-6.283185307179586 upper=6.283185307179586 effort=2.5 velocity=5.76

File: bogobot_rviz/urdf/humanoid_main.urdf.xacro (robot description, xacro)
@@ -2,11 +2,20 @@
 <robot name="Bogobot_V1" xmlns:xacro="http://www.ros.org/wiki/xacro">
     <xacro:include filename="humanoid_links.xacro"/>
+    <!--LINKS-->
+    <!--caja toraxica-->
     <xacro:base_link name="chest" x = "0" y = "0" z = "0.51" row = "0" pitch = "0" yaw = "0"/>
+    <!--brazo izquierdo-->
     <xacro:shoulder_link_base name="link_base_left_shoulder" x = "0.0" y = "-0.0185" z = "0.0" row = "0" pitch = "0" yaw = "0"/>
     <xacro:arm_link name="link_left_arm" x = "0.0" y = "0" z = "-0.082" row = "0" pitch = "0" yaw = "0"/>
     <xacro:palm_link name="link_left_palm" x = "0.0" y = "-0.01" z = "-0.062" row = "0" pitch = "0" yaw = "0"/>
+    <!--brazo derecho-->
     <xacro:shoulder_link_base name="link_base_right_shoulder" x = "0.0" y = "0.0185" z = "0.0" row = "0" pitch = "0" yaw = "${pi}"/>
     <xacro:arm_link name="link_right_arm" x = "0.0" y = "0" z = "-0.082" row = "0" pitch = "0" yaw = "${pi}"/>
     <xacro:palm_link name="link_right_palm" x = "0.0" y = "0.01" z = "-0.062" row = "0" pitch = "0" yaw = "${pi}"/>
+    <!--pierna derecha-->
+    <xacro:hip_metal_link name="link_right_hip_metal" x = "0.0" y = "0.0" z = "-0.0175" row = "0" pitch = "0" yaw = "0"/>
+    <!--pierna izquierda-->
+    <xacro:hip_metal_link name="link_left_hip_metal" x = "0.0" y = "0.0" z = "-0.0175" row = "0" pitch = "0" yaw = "0"/>
+    <!--JOINTS-->
     <!--hombro derecho-->
     <joint name="q1" type="revolute">
@@ -57,35 +66,19 @@
         <limit effort="2.5" lower="${-2*pi}" upper="${2*pi}" velocity="5.76"/>
     </joint>
-    <!--
-    <xacro:motor_28 name="left_motor_arm" x = "0" y = "0" z = "0" row = "0" pitch = "0" yaw = "0"/>
-    <xacro:motor_28 name="right_motor_arm" x = "0" y = "0" z = "0" row = "0" pitch = "0" yaw = "0"/>
-    <xacro:shoulder_link_base name="link_left_shoulder" x = "0.0" y = "0.0" z = "0.0" row = "${pi/2}" pitch = "0" yaw = "0"/>
-    <xacro:shoulder_link_base name="link_right_shoulder" x = "0.0" y = "0.0" z = "0.0" row = "${pi/2}" pitch = "0" yaw = "0"/>
-    <joint name="joint_chest_to_left_motor_shoulder" type="fixed">
-        <axis xyz="0 1 0" />
-        <origin xyz="0 0.0925 0.5714" rpy="0 0 0"/>
-        <parent link="chest"/>
-        <child link="left_motor_arm"/>
-    </joint>
-    <joint name="joint_chest_to_right_motor_shoulder" type="fixed">
-        <axis xyz="0 1 0" />
-        <origin xyz="0 -0.0925 0.5714" rpy="0 0 0"/>
-        <parent link="chest"/>
-        <child link="right_motor_arm"/>
-    </joint>
-    <joint name="q1" type="revolute">
-        <origin rpy="0 0 0" xyz="0 0.04 0.017" />
-        <child link="link_left_shoulder" />
-        <parent link="left_motor_arm" />
-        <axis xyz="0 1 0" />
+    <!--pierna derecha-->
+    <joint name="q7" type="revolute">
+        <origin rpy="0 0 0" xyz="0 0.055 0.3825" />
+        <parent link="chest" />
+        <child link="link_right_hip_metal" />
+        <axis xyz="0 0 1" />
         <limit effort="2.5" lower="${-2*pi}" upper="${2*pi}" velocity="5.76"/>
     </joint>
-    <joint name="q2_b" type="revolute">
-        <origin rpy="0 0 0" xyz="0 -0.04 0.017" />
-        <child link="link_right_shoulder" />
-        <parent link="right_motor_arm" />
-        <axis xyz="0 1 0" />
+    <!--pierna izquierda-->
+    <joint name="q8" type="revolute">
+        <origin rpy="0 0 0" xyz="0 -0.055 0.3825" />
+        <parent link="chest" />
+        <child link="link_left_hip_metal" />
+        <axis xyz="0 0 1" />
         <limit effort="2.5" lower="${-2*pi}" upper="${2*pi}" velocity="5.76"/>
     </joint>
-    -->
 </robot>

Commit message: hip motors added

File: bogobot_rviz/urdf/humanoid_links.xacro (robot description, xacro)
@@ -100,3 +100,19 @@
 		</link>
 	</xacro:macro>
+	<xacro:macro name="motor_double_join" params="name x y z row pitch yaw">
+		<link name="${name}">
+			<collision>
+                		<origin xyz="${x} ${y} ${z}" rpy="${row} ${pitch} ${yaw}"  />
+                		<geometry>
+                    			<mesh filename="package://bogobot_rviz/meshes/motor_doble_join.STL" scale="0.001 0.001 0.001"/>
+                		</geometry>
+            		</collision>
+			<visual>
+                		<origin xyz="${x} ${y} ${z}" rpy="${row} ${pitch} ${yaw}" />
+                		<geometry>
+                    			<mesh filename="package://bogobot_rviz/meshes/motor_doble_join.STL" scale="0.001 0.001 0.001"/>
+                		</geometry>
+            		</visual>
+		</link>
+	</xacro:macro>
 </robot>

File: bogobot_rviz/urdf/humanoid_main.urdf (robot description, URDF)
Before this commit: robot Bogobot_V1, 9 links, 8 joints
Links:
- added link link_left_hip_motor; collision mesh filename=package://bogobot_rviz/meshes/motor_doble_join.STL scale=0.001 0.001 0.001; visual mesh filename=package://bogobot_rviz/meshes/motor_doble_join.STL scale=0.001 0.001 0.001
- added link link_right_hip_motor; collision mesh filename=package://bogobot_rviz/meshes/motor_doble_join.STL scale=0.001 0.001 0.001; visual mesh filename=package://bogobot_rviz/meshes/motor_doble_join.STL scale=0.001 0.001 0.001
Joints:
- added joint q10: type revolute, parent link_left_hip_metal, child link_left_hip_motor, origin xyz=0 0 -0.025 rpy=0 0 0, axis 1 0 0, limit lower=-6.283185307179586 upper=6.283185307179586 effort=2.5 velocity=5.76
- added joint q9: type revolute, parent link_right_hip_metal, child link_right_hip_motor, origin xyz=0 0 -0.025 rpy=0 0 0, axis 1 0 0, limit lower=-6.283185307179586 upper=6.283185307179586 effort=2.5 velocity=5.76
- joint q7: axis 1 0 0 -> 0 0 1
- joint q8: axis 1 0 0 -> 0 0 1

File: bogobot_rviz/urdf/humanoid_main.urdf.xacro (robot description, xacro)
@@ -15,6 +15,8 @@
     <!--pierna derecha-->
     <xacro:hip_metal_link name="link_right_hip_metal" x = "0.0" y = "0.0" z = "-0.0175" row = "0" pitch = "0" yaw = "0"/>
+    <xacro:motor_double_join name="link_right_hip_motor" x = "0.0" y = "0.0" z = "-0.0225" row = "0" pitch = "0" yaw = "0"/>
     <!--pierna izquierda-->
     <xacro:hip_metal_link name="link_left_hip_metal" x = "0.0" y = "0.0" z = "-0.0175" row = "0" pitch = "0" yaw = "0"/>
+    <xacro:motor_double_join name="link_left_hip_motor" x = "0.0" y = "0.0" z = "-0.0225" row = "0" pitch = "0" yaw = "0"/>
     <!--JOINTS-->
     <!--hombro derecho-->
@@ -74,4 +76,11 @@
         <limit effort="2.5" lower="${-2*pi}" upper="${2*pi}" velocity="5.76"/>
     </joint>
+    <joint name="q9" type="revolute">
+        <origin rpy="0 0 0" xyz="0 0 -0.025" />
+        <parent link="link_right_hip_metal" />
+        <child link="link_right_hip_motor" />
+        <axis xyz="1 0 0" />
+        <limit effort="2.5" lower="${-2*pi}" upper="${2*pi}" velocity="5.76"/>
+    </joint>
     <!--pierna izquierda-->
     <joint name="q8" type="revolute">
@@ -82,3 +91,10 @@
         <limit effort="2.5" lower="${-2*pi}" upper="${2*pi}" velocity="5.76"/>
     </joint>
+    <joint name="q10" type="revolute">
+        <origin rpy="0 0 0" xyz="0 0 -0.025" />
+        <parent link="link_left_hip_metal" />
+        <child link="link_left_hip_motor" />
+        <axis xyz="1 0 0" />
+        <limit effort="2.5" lower="${-2*pi}" upper="${2*pi}" velocity="5.76"/>
+    </joint>
 </robot>
